File: power_NAND_2input.brd (EAGLE design)
At the start: 28.9 x 24.3 mm, 17 parts, among them Q1 2n2222, Q2 2n2222, Q3 2n2222, Q4 2n2222, Q5 2n2222, Q6 2n2222

Commit message: new design for power_nand
Parts:
- moved D1 8.89 mm to (75.7, 62.4), turned to 90 degrees
- moved Q5 7.68 mm to (76.8, 68.1), turned to 270 degrees
- moved R1 6.16 mm to (63.1, 77.7)
- moved Q6 5.47 mm to (70.1, 61.7), turned to 180 degrees
- moved R3 4.55 mm to (78.9, 77.7)
- moved Q4 3.07 mm to (76.8, 71.5)
- moved R2 2.56 mm to (76.6, 77.7)
- moved R0 0.92 mm to (73.3, 68.8)
Routing:
- net OUT: track 32.4 -> 20.2 mm
- net N$6: track 20.5 -> 13.1 mm
- net +5V: track 27.3 -> 21.9 mm
- net GND: track 20.5 -> 15.6 mm
- net N$11: track 2.49 -> 5.51 mm
- net N$3: track 6.38 -> 5.04 mm
- net N$4: track 12.3 -> 11.1 mm
- net N$5: track 8.06 -> 9.09 mm
Other:
- board size 28.9 x 24.3 mm -> 24.1 x 21.6 mm
- board text added: "NAND Ver2.1 Alwaro & Gryglu"
- board text removed: "NAND Ver2.0 Alwaro & Gryglu"
